File: arduino-sss.sch (KiCad schematic (older format))
At the start: 47 parts, among them J1 Conn_01x03_Male, J2 Barrel_Jack_Switch, J3 DB9_Male, J4 Conn_01x02_Male, J5 Conn_02x03_Odd_Even, P1 Power, P2 Analog, P3 Digital, P4 Digital, P5 CONN_01X01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

Commit message: update
Parts:
- J3: value DB9_Male -> DB9_Female_MountingHoles; footprint Connector_Dsub:DSUB-9_Male_Horizontal_P2.77x2.54mm_EdgePinOffset9.40mm -> Connector_Dsub:DSUB-9_Female_Horizontal_P2.77x2.84mm_EdgePinOffset4.94mm_Housed_MountingHolesOffset7.48mm; symbol Connector:DB9_Male -> Connector:DB9_Female_MountingHoles
Connections:
- net GNDD: now also J3.0 (PAD)
- no-connect marks 5 -> 10
Changed lines of the file:
@@
 EESchema Schematic File Version 4
 LIBS:arduino-sss-cache
-EELAYER 26 0
+EELAYER 30 0
 EELAYER END
 $Descr A4 11693 8268
@@
 $EndComp
 $Comp
-L Connector:DB9_Male J3
-U 1 1 5C3D621D
-P 2350 4650
-F 0 "J3" H 2270 3958 50  0000 C CNN
-F 1 "DB9_Male" H 2270 4049 50  0000 C CNN
-F 2 "Connector_Dsub:DSUB-9_Male_Horizontal_P2.77x2.54mm_EdgePinOffset9.40mm" H 2350 4650 50  0001 C CNN
-F 3 " ~" H 2350 4650 50  0001 C CNN
-	1    2350 4650
-	-1   0    0    1
-$EndComp
-$Comp
 L power:GNDD #PWR0110
 U 1 1 5C3D8C39
-P 2650 5200
-F 0 "#PWR0110" H 2650 4950 50  0001 C CNN
-F 1 "GNDD" H 2654 5045 50  0000 C CNN
-F 2 "" H 2650 5200 50  0001 C CNN
-F 3 "" H 2650 5200 50  0001 C CNN
-	1    2650 5200
+P 2650 5300
+F 0 "#PWR0110" H 2650 5050 50  0001 C CNN
+F 1 "GNDD" H 2654 5145 50  0000 C CNN
+F 2 "" H 2650 5300 50  0001 C CNN
+F 3 "" H 2650 5300 50  0001 C CNN
+	1    2650 5300
 	1    0    0    -1
 $EndComp
@@
 	1    0    0    -1
 $EndComp
-Wire Wire Line
-	2650 5050 2650 5200
 $Comp
 L Connector:Conn_01x03_Male J1
@@
 $EndComp
 Connection ~ 3250 4650
+NoConn ~ 2650 4250
+NoConn ~ 2650 4350
+NoConn ~ 2650 4550
+NoConn ~ 2650 4750
+NoConn ~ 2650 4950
+$Comp
+L Connector:DB9_Female_MountingHoles J3
+U 1 1 5C3D621D
+P 2350 4650
+F 0 "J3" H 2500 5400 50  0000 C CNN
+F 1 "DB9_Female_MountingHoles" H 2350 5250 50  0000 C CNN
+F 2 "Connector_Dsub:DSUB-9_Female_Horizontal_P2.77x2.84mm_EdgePinOffset4.94mm_Housed_MountingHolesOffset7.48mm" H 2350 4650 50  0001 C CNN
+F 3 " ~" H 2350 4650 50  0001 C CNN
+	1    2350 4650
+	-1   0    0    -1
+$EndComp
+Wire Wire Line
+	2650 5050 2650 5250
+Wire Wire Line
+	2350 5250 2650 5250
+Connection ~ 2650 5250
+Wire Wire Line
+	2650 5250 2650 5300
 $EndSCHEMATC

Commit message: update according to Real BOM
Parts:
- C1, C4: footprint Capacitor_THT:CP_Radial_D4.0mm_P1.50mm -> Capacitor_THT:C_Radial_D5.0mm_H7.0mm_P2.00mm
- C2, C5, C8, C9: footprint Capacitor_THT:C_Axial_L3.8mm_D2.6mm_P7.50mm_Horizontal -> Capacitor_THT:C_Disc_D8.0mm_W5.0mm_P7.50mm
- C3: footprint Capacitor_THT:C_Radial_D4.0mm_H5.0mm_P1.50mm -> Capacitor_THT:C_Radial_D4.0mm_H7.0mm_P1.50mm
- C6, C7: footprint Capacitor_THT:C_Disc_D3.0mm_W1.6mm_P2.50mm -> Capacitor_THT:C_Disc_D5.0mm_W2.5mm_P2.50mm
- D7: value LED13 -> L
- J1: value Conn_01x03_Male -> SERIAL
- J3: footprint Connector_Dsub:DSUB-9_Female_Horizontal_P2.77x2.84mm_EdgePinOffset4.94mm_Housed_MountingHolesOffset7.48mm -> Connector_Dsub:DSUB-9_Female_Horizontal_P2.77x2.84mm_EdgePinOffset7.70mm_Housed_MountingHolesOffset9.12mm
- J4: value Conn_01x02_Male -> AUTO RESET
- J5: value Conn_02x03_Odd_Even -> ICSP
- L1: footprint Inductor_THT:L_Axial_L5.0mm_D3.6mm_P10.00mm_Horizontal_Murata_BL01RN1A2A2 -> Inductor_THT:L_Axial_L12.0mm_D5.0mm_P15.24mm_Horizontal_Fastron_MISC
- Q1, Q2: footprint Package_TO_SOT_THT:TO-92_Inline -> Package_TO_SOT_THT:TO-92_Inline_Wide
- U2: footprint Package_DIP:DIP-28_W7.62mm -> Package_DIP:DIP-28_W7.62mm_Socket
- Y1: footprint Crystal:Crystal_HC18-U_Horizontal -> Crystal:Crystal_HC49-4H_Vertical
Changed lines of the file:
@@
 F 0 "C1" H 2568 1146 50  0000 L CNN
 F 1 "100u" H 2568 1055 50  0000 L CNN
-F 2 "Capacitor_THT:CP_Radial_D4.0mm_P1.50mm" H 2488 950 50  0001 C CNN
+F 2 "Capacitor_THT:C_Radial_D5.0mm_H7.0mm_P2.00mm" H 2488 950 50  0001 C CNN
 F 3 "~" H 2450 1100 50  0001 C CNN
 	1    2450 1100
@@
 F 0 "C2" H 2965 1146 50  0000 L CNN
 F 1 "100n" H 2965 1055 50  0000 L CNN
-F 2 "Capacitor_THT:C_Axial_L3.8mm_D2.6mm_P7.50mm_Horizontal" H 2888 950 50  0001 C CNN
+F 2 "Capacitor_THT:C_Disc_D8.0mm_W5.0mm_P7.50mm" H 2888 950 50  0001 C CNN
 F 3 "~" H 2850 1100 50  0001 C CNN
 	1    2850 1100
@@
 F 0 "C4" H 4118 1146 50  0000 L CNN
 F 1 "100u" H 4118 1055 50  0000 L CNN
-F 2 "Capacitor_THT:CP_Radial_D4.0mm_P1.50mm" H 4038 950 50  0001 C CNN
+F 2 "Capacitor_THT:C_Radial_D5.0mm_H7.0mm_P2.00mm" H 4038 950 50  0001 C CNN
 F 3 "~" H 4000 1100 50  0001 C CNN
 	1    4000 1100
@@
 P 1350 4550
 F 0 "J1" V 1410 4690 50  0000 L CNN
-F 1 "Conn_01x03_Male" V 1501 4690 50  0000 L CNN
+F 1 "SERIAL" V 1501 4690 50  0000 L CNN
 F 2 "Connector_PinHeader_2.54mm:PinHeader_1x03_P2.54mm_Vertical" H 1350 4550 50  0001 C CNN
 F 3 "~" H 1350 4550 50  0001 C CNN
@@
 F 0 "Q1" H 3391 6696 50  0000 L CNN
 F 1 "BC547" H 3391 6605 50  0000 L CNN
-F 2 "Package_TO_SOT_THT:TO-92_Inline" H 3400 6575 50  0001 L CIN
+F 2 "Package_TO_SOT_THT:TO-92_Inline_Wide" H 3400 6575 50  0001 L CIN
 F 3 "http://www.fairchildsemi.com/ds/BC/BC547.pdf" H 3200 6650 50  0001 L CNN
 	1    3200 6650
@@
 F 0 "Q2" H 3540 3904 50  0000 L CNN
 F 1 "BC557" H 3540 3995 50  0000 L CNN
-F 2 "Package_TO_SOT_THT:TO-92_Inline" H 3550 3875 50  0001 L CIN
+F 2 "Package_TO_SOT_THT:TO-92_Inline_Wide" H 3550 3875 50  0001 L CIN
 F 3 "http://www.fairchildsemi.com/ds/BC/BC557.pdf" H 3350 3950 50  0001 L CNN
 	1    3350 3950
@@
 F 0 "U2" H 7800 6328 50  0000 C CNN
 F 1 "ATmega8-16PU" H 7800 6237 50  0000 C CNN
-F 2 "Package_DIP:DIP-28_W7.62mm" H 7800 4750 50  0001 C CIN
+F 2 "Package_DIP:DIP-28_W7.62mm_Socket" H 7800 4750 50  0001 C CIN
 F 3 "http://ww1.microchip.com/downloads/en/DeviceDoc/atmel-2486-8-bit-avr-microcontroller-atmega8_l_datasheet.pdf" H 7800 4750 50  0001 C CNN
 	1    7800 4750
@@
 P 5150 3450
 F 0 "J4" V 5210 3490 50  0000 L CNN
-F 1 "Conn_01x02_Male" V 5301 3490 50  0000 L CNN
+F 1 "AUTO RESET" V 5301 3490 50  0000 L CNN
 F 2 "Connector_PinHeader_2.54mm:PinHeader_1x02_P2.54mm_Vertical" H 5150 3450 50  0001 C CNN
 F 3 "~" H 5150 3450 50  0001 C CNN
@@
 F 0 "C5" H 4765 4396 50  0000 L CNN
 F 1 "100n" H 4765 4305 50  0000 L CNN
-F 2 "Capacitor_THT:C_Axial_L3.8mm_D2.6mm_P7.50mm_Horizontal" H 4688 4200 50  0001 C CNN
+F 2 "Capacitor_THT:C_Disc_D8.0mm_W5.0mm_P7.50mm" H 4688 4200 50  0001 C CNN
 F 3 "~" H 4650 4350 50  0001 C CNN
 	1    4650 4350
@@
 P 6300 2450
 F 0 "J5" H 6350 2767 50  0000 C CNN
-F 1 "Conn_02x03_Odd_Even" H 6350 2676 50  0000 C CNN
+F 1 "ICSP" H 6350 2676 50  0000 C CNN
 F 2 "Connector_PinHeader_2.54mm:PinHeader_2x03_P2.54mm_Vertical" H 6300 2450 50  0001 C CNN
 F 3 "~" H 6300 2450 50  0001 C CNN
@@
 F 0 "Y1" V 6554 4081 50  0000 L CNN
 F 1 "16000" V 6645 4081 50  0000 L CNN
-F 2 "Crystal:Crystal_HC18-U_Horizontal" H 6600 3950 50  0001 C CNN
+F 2 "Crystal:Crystal_HC49-4H_Vertical" H 6600 3950 50  0001 C CNN
 F 3 "~" H 6600 3950 50  0001 C CNN
 	1    6600 3950
@@
 F 0 "C6" V 6048 3800 50  0000 C CNN
 F 1 "22p" V 6139 3800 50  0000 C CNN
-F 2 "Capacitor_THT:C_Disc_D3.0mm_W1.6mm_P2.50mm" H 6338 3650 50  0001 C CNN
+F 2 "Capacitor_THT:C_Disc_D5.0mm_W2.5mm_P2.50mm" H 6338 3650 50  0001 C CNN
 F 3 "~" H 6300 3800 50  0001 C CNN
 	1    6300 3800
@@
 F 0 "C7" V 6048 4100 50  0000 C CNN
 F 1 "22p" V 6139 4100 50  0000 C CNN
-F 2 "Capacitor_THT:C_Disc_D3.0mm_W1.6mm_P2.50mm" H 6338 3950 50  0001 C CNN
+F 2 "Capacitor_THT:C_Disc_D5.0mm_W2.5mm_P2.50mm" H 6338 3950 50  0001 C CNN
 F 3 "~" H 6300 4100 50  0001 C CNN
 	1    6300 4100
@@
 F 0 "L1" V 7854 3127 50  0000 L CNN
 F 1 "100u" V 7945 3127 50  0000 L CNN
-F 2 "Inductor_THT:L_Axial_L5.0mm_D3.6mm_P10.00mm_Horizontal_Murata_BL01RN1A2A2" H 7900 3050 50  0001 C CNN
+F 2 "Inductor_THT:L_Axial_L12.0mm_D5.0mm_P15.24mm_Horizontal_Fastron_MISC" H 7900 3050 50  0001 C CNN
 F 3 "~" H 7900 3050 50  0001 C CNN
 	1    7900 3050
@@
 F 0 "C9" V 7898 3350 50  0000 C CNN
 F 1 "100n" V 7989 3350 50  0000 C CNN
-F 2 "Capacitor_THT:C_Axial_L3.8mm_D2.6mm_P7.50mm_Horizontal" H 8188 3200 50  0001 C CNN
+F 2 "Capacitor_THT:C_Disc_D8.0mm_W5.0mm_P7.50mm" H 8188 3200 50  0001 C CNN
 F 3 "~" H 8150 3350 50  0001 C CNN
 	1    8150 3350
@@
 F 0 "C8" V 7898 2800 50  0000 C CNN
 F 1 "100n" V 7989 2800 50  0000 C CNN
-F 2 "Capacitor_THT:C_Axial_L3.8mm_D2.6mm_P7.50mm_Horizontal" H 8188 2650 50  0001 C CNN
+F 2 "Capacitor_THT:C_Disc_D8.0mm_W5.0mm_P7.50mm" H 8188 2650 50  0001 C CNN
 F 3 "~" H 8150 2800 50  0001 C CNN
 	1    8150 2800
@@
 P 9000 4150
 F 0 "D7" V 9038 4032 50  0000 R CNN
-F 1 "LED13" V 8947 4032 50  0000 R CNN
+F 1 "L" V 8947 4032 50  0000 R CNN
 F 2 "LED_THT:LED_D3.0mm_Clear" H 9000 4150 50  0001 C CNN
 F 3 "~" H 9000 4150 50  0001 C CNN
@@
 F 0 "C3" H 3365 4846 50  0000 L CNN
 F 1 "10u" H 3365 4755 50  0000 L CNN
-F 2 "Capacitor_THT:C_Radial_D4.0mm_H5.0mm_P1.50mm" H 3288 4650 50  0001 C CNN
+F 2 "Capacitor_THT:C_Radial_D4.0mm_H7.0mm_P1.50mm" H 3288 4650 50  0001 C CNN
 F 3 "~" H 3250 4800 50  0001 C CNN
 	1    3250 4800
@@
 F 0 "J3" H 2500 5400 50  0000 C CNN
 F 1 "DB9_Female_MountingHoles" H 2350 5250 50  0000 C CNN
-F 2 "Connector_Dsub:DSUB-9_Female_Horizontal_P2.77x2.84mm_EdgePinOffset4.94mm_Housed_MountingHolesOffset7.48mm" H 2350 4650 50  0001 C CNN
+F 2 "Connector_Dsub:DSUB-9_Female_Horizontal_P2.77x2.84mm_EdgePinOffset7.70mm_Housed_MountingHolesOffset9.12mm" H 2350 4650 50  0001 C CNN
 F 3 " ~" H 2350 4650 50  0001 C CNN
 	1    2350 4650
